File: io-board/LED_Driver.kicad_sch (KiCad schematic)
At the start: 15 parts, among them Q12 NPN, Q13 PNP

Commit message: PCB: io: Removed unneeded res in LED driver
Parts:
- removed R42: R, Resistor_SMD:R_0805_2012Metric_Pad1.20x1.40mm_HandSolder, symbol Device:R
Connections:
- net at R40.2, R41.1: now also Q13.1 (B)
Changed lines of the file:
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@@
 	(wire
 		(pts
-			(xy 124.46 91.44) (xy 127 91.44)
+			(xy 124.46 91.44) (xy 137.16 91.44)
 		)
 		(stroke
@@
 		(pts
 			(xy 114.3 107.95) (xy 116.84 107.95)
-		)
-		(stroke
-			(width 0)
-			(type default)
-		)
-	)
-	(wire
-		(pts
-			(xy 134.62 91.44) (xy 137.16 91.44)
 		)
 		(stroke
@@
 					(unit 1)
 				)
-			)
-		)
-	)
-	(symbol
-		(lib_id "Device:R")
-		(at 130.81 91.44 90)
-		(unit 1)
-		(exclude_from_sim no)
-		(in_bom yes)
-		(on_board yes)
-		(dnp no)
-		(property "Reference" "R42"
-			(at 132.334 89.408 90)
-			(effects
-				(font
-					(size 1.27 1.27)
-				)
-			)
-		)
-		(property "Value" "R"
-			(at 129.032 89.408 90)
-			(effects
-				(font
-					(size 1.27 1.27)
-				)
-				(hide yes)
-			)
-		)
-		(property "Footprint" "Resistor_SMD:R_0805_2012Metric_Pad1.20x1.40mm_HandSolder"
-			(at 130.81 93.218 90)
-			(effects
-				(font
-					(size 1.27 1.27)
-				)
-				(hide yes)
-			)
-		)
-		(property "Datasheet" "~"
-			(at 130.81 91.44 0)
-			(effects
-				(font
-					(size 1.27 1.27)
-				)
-				(hide yes)
-			)
-		)
-		(property "Description" "Resistor"
-			(at 130.81 91.44 0)
-			(effects
-				(font
-					(size 1.27 1.27)
-				)
-				(hide yes)
-			)
-		)
-		(pin "2"
-		)
-		(pin "1"
-		)
-		(instances
-			(project "io-board"
-				(path "/5a6848ff-426f-432e-bc4d-b6eef5e4348a/5680163a-59ef-49fe-bd7d-0718bd629dd1"
-					(reference "R42")
-					(unit 1)
-				)
-				(path "/5a6848ff-426f-432e-bc4d-b6eef5e4348a/e46419f4-efe2-457e-998d-7494f8c6e183"
-					(reference "R50")
-					(unit 1)
-				)

Commit message: PCB: io-board: component values and BOM
Parts:
- C20, C21: value C -> 47uF
- D12, D13, D14: value D -> Vishay MCL4448-TR
- Q12: value NPN -> NPN BC847C-AQ
- Q13: value PNP -> PNP BC857C-AQ
- R39, R40, R41, R44: value R -> 2.2K
- R43, R45: value R -> 68
- R46: value R -> 100
Other:
- note added: "WARNING!!! Connected to GND"
Changed lines of the file:
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@@
 	(generator_version "9.0")
 	(paper "A4")
+	(text "WARNING!!!\nConnected to GND"
+		(exclude_from_sim no)
+		(at 156.972 72.898 0)
+		(effects
+			(font
+				(size 1.27 1.27)
+			)
+		)
+	)
+	(text_box "TODO:\n* PIN ADC jest 5V tolerant, jeżeli nie, to zmiejszyć mapięcie na drabince rezystorów\n* Rezystor rozładowujący powinien być podłączony do masy.\n  Wtedy jest łatwa detekcja rozłączenia LED - jest ~0V na ADC.\n  Jeżeli tak jest, to PWM się wyłącza. TODO: algorytm ponownego włączenia.\n  \n\nhttps ://www.falstad.com/circuit/circuitjs.html?ctz=CQAgjCAMB0l3EDMAOATNA7ANlQVjWACyICcJkWhIuG11k1ApgLRhgBQA5tSatWH1y9qqZFCjsAxjz7FBw3AJBUY8SCRXjI7AE4hEiLMsSy4xvg1Tx2ABxDIzhQmIcNFfRFokA3fYf4e-nLigvDg0LjhkQyqiFx+Ru4J1FgxEgAuyo4mypTm4hBpYGYAJowAZgCGAK4ANunxhHlOYk1UhCRGMbq57WBGbfq4FiBWcD2DiMO9o8hiltYASjOirXl4XeKEDEppMLjsmbhOQ-Ie0wysXsUMZVV1DctCgYnCG17b4CMxET0Y0y0QP9BLsQFhkOx+nw2JAqKhUFQYVRELDRiA7jV6sxaowSuAvKoOFDwMVkaikfpkHD0RVMelsbj8XtYBw9M98uzDPMwRDuMCAkDpsNudo9BhUSgqPzViExuwAO72RzOQWyFXaRX8pKuAUamT5LAYWQ5PWG418M2UlQKsFGq22vgy012mXSuYSTXTSX2PLevWdSzuinw62K5C+qkk1GDUWq5Qq-l+8DjT2O906p2QnBR5GRimDPgYh4MvGFLQs9jbTzhqjCnNgz4MFEAfUozcgzYEohI7dgCF78DAzdYzdQzZbcUVwYRXzMJm6U9J9oEc-BEgAzrOm2uV02rAUQFVauvGDbJkKTlMLJXIJ4wMIBK1+rNuYRm2+O9sSMhm7gB7eBD-EcxzfOJNzmQMxADF8vCPE8b08DpElSBsGEoIpWw-d91B-KxezHYDO3HeJxVzKVo2fBclUg+wHBg7QAHt8TLR9bygPtIEKDiy2hfR2CYsBqwKeESC4wd2PEiBoU8OIgA"
+		(exclude_from_sim no)
+		(at 220.98 134.62 0)
+		(size 62.23 29.21)
+		(margins 0.9525 0.9525 0.9525 0.9525)
+		(stroke
+			(width 0)
+			(type solid)
+		)
+		(fill
+			(type none)
+		)
+		(effects
+			(font
+				(size 0.762 0.762)
+			)
+			(justify left top)
+		)
+	)
 	(junction
 		(at 152.4 111.76)
@@
 		)
 	)
+	(polyline
+		(pts
+			(xy 167.64 88.9) (xy 170.18 88.9)
+		)
+		(stroke
+			(width 0)
+			(type default)
+		)
+	)
 	(wire
 		(pts
@@
 		)
 	)
+	(polyline
+		(pts
+			(xy 167.64 74.93) (xy 167.64 88.9)
+		)
+		(stroke
+			(width 0)
+			(type default)
+		)
+	)
 	(wire
 		(pts
@@
 		(pts
 			(xy 184.15 101.6) (xy 184.15 116.84)
+		)
+		(stroke
+			(width 0)
+			(type default)
+		)
+	)
+	(polyline
+		(pts
+			(xy 148.59 74.93) (xy 167.64 74.93)
 		)
 		(stroke
@@
 		(on_board yes)
 		(dnp no)
-		(fields_autoplaced yes)
 		(property "Reference" "Q12"
 			(at 127 106.6799 0)
@@
 			)
 		)
-		(property "Value" "NPN"
-			(at 127 109.2199 0)
+		(property "Value" "NPN BC847C-AQ"
+			(at 117.602 113.538 0)
 			(effects
 				(font
@@
 			)
 		)
-		(property "Value" "R"
-			(at 169.418 112.268 90)
-			(effects
-				(font
-					(size 1.27 1.27)
-				)
-				(hide yes)
+		(property "Value" "68"
+			(at 173.99 109.728 90)
+			(effects
+				(font
+					(size 1.27 1.27)
+				)
 			)
 		)
@@
 			)
 		)
-		(property "Value" "R"
-			(at 122.428 98.298 90)
-			(effects
-				(font
-					(size 1.27 1.27)
-				)
-				(hide yes)
+		(property "Value" "2.2K"
+			(at 127.254 96.52 90)
+			(effects
+				(font
+					(size 1.27 1.27)
+				)
 			)
 		)
@@
 			)
 		)
-		(property "Value" "D"
+		(property "Value" "Vishay MCL4448-TR"
 			(at 186.69 86.3599 90)
 			(effects
@@
 			)
 		)
-		(property "Value" "R"
-			(at 108.712 105.918 90)
-			(effects
-				(font
-					(size 1.27 1.27)
-				)
-				(hide yes)
+		(property "Value" "2.2K"
+			(at 110.236 110.49 90)
+			(effects
+				(font
+					(size 1.27 1.27)
+				)
 			)
 		)
@@
 			)
 		)
-		(property "Value" "D"
+		(property "Value" "Vishay MCL4448-TR"
 			(at 186.69 99.0599 90)
 			(effects
@@
 			)
 		)
-		(property "Value" "C"
-			(at 156.21 109.2199 0)
+		(property "Value" "47uF"
+			(at 153.67 110.49 0)
 			(effects
 				(font
@@
 				)
 				(justify left)
-				(hide yes)
 			)
 		)
@@
 			)
 		)
-		(property "Value" "R"
-			(at 169.418 99.568 90)
-			(effects
-				(font
-					(size 1.27 1.27)
-				)
-				(hide yes)
+		(property "Value" "100"
+			(at 173.99 97.282 90)
+			(effects
+				(font
+					(size 1.27 1.27)
+				)
 			)
 		)
@@
 			)
 		)
-		(property "Value" "C"
-			(at 148.59 109.2199 0)
+		(property "Value" "47uF"
+			(at 139.192 110.998 0)
 			(effects
 				(font
@@
 				)
 				(justify left)
-				(hide yes)
 			)
 		)
@@
 			)
 		)
-		(property "Value" "R"
-			(at 142.748 102.108 90)
-			(effects
-				(font
-					(size 1.27 1.27)
-				)
-				(hide yes)
+		(property "Value" "68"
+			(at 147.066 98.552 90)
+			(effects
+				(font
+					(size 1.27 1.27)
+				)
 			)
 		)
@@
 			)
 		)
-		(property "Value" "R"
-			(at 122.428 88.138 90)
-			(effects
-				(font
-					(size 1.27 1.27)
-				)
-				(hide yes)
+		(property "Value" "2.2K"
+			(at 127 86.106 90)
+			(effects
+				(font
+					(size 1.27 1.27)
+				)
 			)
 		)
@@
 			)
 		)
-		(property "Value" "R"
-			(at 169.418 86.868 90)
-			(effects
-				(font
-					(size 1.27 1.27)
-				)
-				(hide yes)
+		(property "Value" "2.2K"
+			(at 174.498 85.344 90)
+			(effects
+				(font
+					(size 1.27 1.27)
+				)
 			)
 		)
@@
 			)
 		)
-		(property "Value" "D"
+		(property "Value" "Vishay MCL4448-TR"
 			(at 186.69 77.4699 90)
 			(effects
@@
 		(on_board yes)
 		(dnp no)
-		(fields_autoplaced yes)
 		(property "Reference" "Q13"
 			(at 147.32 92.7101 0)
@@
 			)
 		)
-		(property "Value" "PNP"
-			(at 147.32 90.1701 0)
-			(effects
-				(font
+		(property "Value" "PNP BC857C-AQ"
+			(at 138.176 85.344 0)
+			(effects
+				(font
