File: comm-board-ext-router/comm-board-ext-router.kicad_sch (KiCad schematic)
At the start: 42 parts, among them J1 GND - DC-DC, J10 MCU-RxD1, J11 MCU-TxD2, J12 MCU-RxD2, J14 Board - 5V, J15 Board - 12V, J17 Board - GND, J2 GND - DC-DC, J25 MID1 - Board, J28 Board - 3.3V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

Commit message: comm-board: New "Gateway" and "Router" extensions and removed old "Universal"
Parts:
- removed C1: C, Footprints:CNC-mill-0.7-CAP, symbol Device:C
- removed D1, D2: D, Footprints:CNC-mill-0.7-RES, symbol Device:D
- removed R3, R4: R, Footprints:CNC-mill-0.7-RES, symbol Device:R
- removed R5: 0, Footprints:CNC-mill-0.7-RES, symbol Device:R
- added J27, J30: ~, Footprints:VHDR, symbol Connector_Generic:Conn_01x01
- R1, R2, R7, R8: value R -> 3.3K
- U1, U2: footprint Footprints:CNC-mill-0.7-DIP-8 -> Footprints:CNC-mill-0.8-DIP-8
Connections:
- net +5V: now also R1.1; no longer J22.1 (Pin_1), J23.1 (Pin_1)
- net GND: now also R2.2, J27.1 (Pin_1), J30.1 (Pin_1)
- net RxD2: now also J22.1 (Pin_1), J23.1 (Pin_1)
- net at J29.1 (Pin_1), R2.1: now also R1.2
- net at R7.2, R8.1: now also J25.1 (Pin_1); no longer R1.1, R2.2
Other:
- note removed: "1-wire UART alternative"
- note removed: "R-Pi alternative"
- moved on the sheet: J25, J29, R1, R2
